File: hardware/kicad/th_sensor_h2.kicad_sch (KiCad schematic)
At the start: 74 parts, among them J1 DEBUG, Q1 AO3401A, Q2 AO3401A, Q3 2N7002, Q4 2N7002, SW1 USER/BOOT, SW2 RST, U1 TPS63900DSKR, U2 TPS63900DSKR, U3 TPS3839K33DBZR, U4 ESP32-H2-MINI-1-H4S, U5 SHT40-AD1B-R3, Y1 32.768kHz

Commit message: Route the PCB with a scripted grid router; move module per antenna guide
- Module moved to the top-left corner (<= 2 mm from the edge) with a
  15 mm board notch beside the antenna, per the ESP32-H2 hardware design
  guidelines keepout figure. The left edge now carries only 3V3 and EN,
  so VBAT_MEAS_EN moves to GPIO12, VBAT1_SENSE to GPIO5 (ADC1_CH4) and
  the LED to GPIO22 (schematic, firmware pin map and ADC channel).
- J1 becomes a horizontal 1x7 header under the notch, ordered like the
  module pins; EN is no longer on the header.
- gen_pcb.py: converter blocks laid out after the TPS63900 datasheet
  example with hand-routed power loops, fixed SHT40 tongue routing,
  module escape stubs, GND fanout, planes, stitching vias.
- router.py: two-layer A* on a 0.1 mm lattice with inflated occupancy
  maps for clearance, turn penalties, via and hole-to-hole checks.

Co-Authored-By: Claude Opus 5.5 <noreply@anthropic.com>
Claude-Session: https://claude.ai/code/session_01TvrXHUQLozvfXGbtsTcbbw
Parts:
- J1: footprint Connector_PinHeader_2.54mm:PinHeader_1x08_P2.54mm_Vertical -> Connector_PinHeader_2.54mm:PinHeader_1x07_P2.54mm_Vertical; symbol Connector_Generic:Conn_01x08 -> Connector_Generic:Conn_01x07
Connections:
- net 3V3_DBG: now also J1.6 (Pin_6); no longer J1.1 (Pin_1)
- net BTN_USER: now also J1.5 (Pin_5); no longer J1.7 (Pin_7)
- net EN: no longer J1.6 (Pin_6)
- net GND: now also J1.7 (Pin_7); no longer J1.8 (Pin_8)
- net LED: now also U4.24 (GPIO22); no longer U4.16 (GPIO12)
- net U0RXD: now also J1.2 (Pin_2); no longer J1.3 (Pin_3)
- net U0TXD: now also J1.1 (Pin_1); no longer J1.2 (Pin_2)
- net USB_DM_J: now also J1.4 (Pin_4); no longer J1.5 (Pin_5)
- net USB_DP_J: now also J1.3 (Pin_3); no longer J1.4 (Pin_4)
- net VBAT1_SENSE: now also U4.19 (GPIO5/FSPID/ADC1_CH4/MTDI); no longer U4.10 (GPIO1/FSPICS0/ADC1_CH0)
- net VBAT_MEAS_EN: now also U4.16 (GPIO12); no longer U4.9 (GPIO0/FSPIQ)
Other:
- note added: "GPIO8/GPIO9 are strapping pins: GPIO9 low at reset (SW1 held) = download mode. VBAT (pad 15) is tied to 3V3 inside the module (R2 = 0R); connected here as well. Unused GPIO0/1/2/3/25: no connect, firmware disables input + pull-down. J1 is a pad row (not fitted): pin 6 3V3_DBG only reaches the rail when JP1 is closed. Reset for programming: SW2 (RST) or the USB-Serial/JTAG reset; EN is not on J1."
- note removed: "GPIO8/GPIO9 are strapping pins: GPIO9 low at reset (SW1 held) = download mode. VBAT (pad 15) is tied to 3V3 inside the module (R2 = 0R); connected here as well. Unused GPIO2/3/5/22/25: no connect, firmware disables input + pull-down. J1 is a pad row (not fitted): pin 1 3V3_DBG only reaches the rail when JP1 is closed."

Commit message: Add EN test pad and net-name test pad labels; reproducible PCB output
Hardware
- TP11 on EN next to the reset button (schematic + PCB); TP9 (GND) moved
  to make room. Schematic: split the EN wire at the new T so kicad-cli
  connects it; fix stale notes (GPIO12 enables the dividers, EN is on
  TP11, not on J1).
- Silkscreen: every test pad shows its net name (VBAT1, VBAT2, VIN1/2,
  VOUT1/2, 3V3_PWR, 3V3, GND, EN); TP numbers stay on the fab drawing.
  "NO CHARGE" under "CR2032 ONLY" as specified, "USER/BOOT" at SW1,
  R1/R11/R21 current links labelled first. Missing required labels now
  stop the generator instead of being dropped.
- gen_pcb.py seeds KiCad's UUID generator, so regenerating gives a
  byte-identical board (KiCad saves items sorted by UUID).
- ERC 0, DRC 0 violations / 0 unconnected / 0 parity errors.

Firmware
- `status` prints free and minimum free heap (bring-up test T-17).

Docs
- README with status table, build/flash/regeneration steps.
- Test plan, architecture, decisions, pin map, assembly, limitations
  updated for TP11, the silkscreen labels, the VBAT_OR equivalence,
  the prod overlay build and disabled secure boot / flash encryption.

Co-Authored-By: Claude Opus 5.5 <noreply@anthropic.com>
Claude-Session: https://claude.ai/code/session_01TvrXHUQLozvfXGbtsTcbbw
Parts:
- added TP11: EN, TestPoint:TestPoint_Pad_D1.5mm, symbol Connector:TestPoint
Connections:
- net EN: now also TP11.1
Other:
- note added: "CR2032 ONLY - NOT RECHARGEABLE. Both cells must be the same brand/lot and replaced together. Power-path decision and its limits: docs/decisions.md, docs/power_budget.md (ESTIMATE until measured). Current measurement: remove R1 / R11 (per cell) or R21 (load) and insert the ammeter. U3 TPS3839K33: 2.93 V typ (2.857-2.974 V), push-pull ~RESET, 200 ms delay; R22 keeps it from fighting SW2 / TP11 (EN)."
- note added: "GPIO8/GPIO9 are strapping pins: GPIO9 low at reset (SW1 held) = download mode. VBAT (pad 15) is tied to 3V3 inside the module (R2 = 0R); connected here as well. Unused GPIO0/1/2/3/25: no connect, firmware disables input + pull-down. J1 is a pad row (not fitted): pin 6 3V3_DBG only reaches the rail when JP1 is closed. Reset for programming: SW2 (RST) or the USB-Serial/JTAG reset; EN is on test pad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"
- note added: "Switches open: no divider current. GPIO12 high for ~30 ms every 6 h: 470k/470k -> 3.3 uA per cell. Each divider top is at the holder terminal (before the 0R link), so a missing cell reads ~0 V."
- note removed: "CR2032 ONLY - NOT RECHARGEABLE. Both cells must be the same brand/lot and replaced together. Power-path decision and its limits: docs/decisions.md, docs/power_budget.md (ESTIMATE until measured). Current measurement: remove R1 / R11 (per cell) or R21 (load) and insert the ammeter. U3 TPS3839K33: 2.93 V typ (2.857-2.974 V), push-pull ~RESET, 200 ms delay; R22 keeps it from fighting SW2 / J1 EN."
- note removed: "GPIO8/GPIO9 are strapping pins: GPIO9 low at reset (SW1 held) = download mode. VBAT (pad 15) is tied to 3V3 inside the module (R2 = 0R); connected here as well. Unused GPIO0/1/2/3/25: no connect, firmware disables input + pull-down. J1 is a pad row (not fitted): pin 6 3V3_DBG only reaches the rail when JP1 is closed. Reset for programming: SW2 (RST) or the USB-Serial/JTAG reset; EN is not on J1."
- note removed: "Switches open: no divider current. GPIO0 high for ~30 ms every 6 h: 470k/470k -> 3.3 uA per cell. Each divider top is at the holder terminal (before the 0R link), so a missing cell reads ~0 V."

Commit message: Rev B: one CR2450, 41.5 x 57.5 mm board
Power path: one CR2450 in an SMT holder (MYOUNG BS-24-B4AA016) ->
0R link -> AO3401A reverse-polarity FET -> one TPS63900 at 3.3 V
(SEL = GND, RCFG3 16.2k; 100 mA input limit) -> VOUT -> 0R link ->
+3V3. No output diode: the cell is the only source. Input buffer
10 uF + 2 x 100 uF MLCC + 470 uF electrolytic. J1 shrinks to 1x6 pads
without a supply pin; test pads VBAT, VIN, VOUT, 3V3, GND, EN.

Board: 72 x 58 mm -> 41.5 x 57.5 mm, holder along the bottom edge,
converter block rotated 180 degrees, SHT40 tongue cut free by one
L-shaped slot. 0 unrouted, ERC/DRC/parity 0; the pours are refilled
under the final project rules before the board is saved.
Silkscreen: front "CR2450 ONLY / NO CHARGE" above the holder, label
placer follows arcs instead of their bounding boxes and tries finer
offsets; R1/R21 link labels are now required.

Firmware: one VBAT channel (GPIO5 / ADC1_CH4), BAT_CELL_COUNT 1,
Power Source reports 1 x CR2450 (620 mAh), single-cell logs/status,
host tests and check_pinmap updated.

Power model: architecture S (one cell); CR2450 resistance scaled
from the CR2032 fit by electrode area (ESTIMATE, bounds x0.4/x1.0).
JLC parts snapshot refreshed 2026-10-30 06:47 UTC.

Co-Authored-By: Claude Opus 5.5 <noreply@anthropic.com>
Claude-Session: https://claude.ai/code/session_01TvrXHUQLozvfXGbtsTcbbw
Parts:
- removed BT2: CR2032 holder, Battery:BatteryHolder_Keystone_1060_1x2032, symbol Device:Battery_Cell
- removed C11: 10uF, Capacitor_SMD:C_0603_1608Metric, symbol Device:C
- removed C12, C13: 100uF, Capacitor_SMD:C_1206_3216Metric, symbol Device:C
- removed C14: 22uF, Capacitor_SMD:C_0805_2012Metric, symbol Device:C
- removed C32: 22nF, Capacitor_SMD:C_0603_1608Metric, symbol Device:C
- removed D1, D2: B5819W, Diode_SMD:D_SOD-123, symbol Device:D_Schottky
- removed J1: DEBUG, Connector_PinHeader_2.54mm:PinHeader_1x07_P2.54mm_Vertical, symbol Connector_Generic:Conn_01x07
- removed JP1: DEBUG_PWR, Jumper:SolderJumper-2_P1.3mm_Open_RoundedPad1.0x1.5mm, symbol Jumper:SolderJumper_2_Open
- removed L2: 2.2uH, th_sensor:L_Murata_DFE201612E, symbol Device:L
- removed Q2: AO3401A, Package_TO_SOT_SMD:SOT-23, symbol th_sensor:AO3401A
- removed Q4: 2N7002, Package_TO_SOT_SMD:SOT-23, symbol th_sensor:2N7002
- removed R11: 0R, Resistor_SMD:R_0805_2012Metric, symbol Device:R
- removed R12: 0R, Resistor_SMD:R_0603_1608Metric, symbol Device:R
- removed R13: 10.5k, Resistor_SMD:R_0603_1608Metric, symbol Device:R
- removed R14: 16.2k, Resistor_SMD:R_0603_1608Metric, symbol Device:R
- removed R33, R34: 470k, Resistor_SMD:R_0603_1608Metric, symbol Device:R
- removed TP10, TP9: GND, TestPoint:TestPoint_Pad_D1.5mm, symbol Connector:TestPoint
- removed TP11: EN, TestPoint:TestPoint_Pad_D1.5mm, symbol Connector:TestPoint
- removed TP7: 3V3_PWR, TestPoint:TestPoint_Pad_D1.5mm, symbol Connector:TestPoint
- removed TP8: 3V3, TestPoint:TestPoint_Pad_D1.5mm, symbol Connector:TestPoint
- removed U2: TPS63900DSKR, Package_SON:WSON-10-1EP_2.5x2.5mm_P0.5mm_EP1.2x2mm, symbol Regulator_Switching:TPS63900
- added C5: 470uF, Capacitor_SMD:CP_Elec_6.3x7.7, symbol Device:C_Polarized
- added J1: DEBUG, Connector_PinHeader_2.54mm:PinHeader_1x06_P2.54mm_Vertical, symbol Connector_Generic:Conn_01x06
- BT1: value CR2032 holder -> CR2450 holder; footprint Battery:BatteryHolder_Keystone_1060_1x2032 -> th_sensor:BatteryHolder_MYOUNG_BS-24-B4AA016_1x2450; LCSC C238069 -> C964809; MPN 1060TR -> BS-24-B4AA016; Manufacturer Keystone -> MYOUNG
- TP1: value VBAT1 -> VBAT
- TP2: value VBAT2 -> VIN
- TP3: value VIN1 -> VOUT
- TP4: value VIN2 -> 3V3
- TP5: value VOUT1 -> GND
- TP6: value VOUT2 -> EN
Connections:
- net VIN2 is gone; now on net +3V3: TP4.1
- net VOUT2 is gone; now on net EN: TP6.1
- net BTN_USER: now also J1.5 (Pin_5)
- net GND: now also TP5.1, U1.2 (SEL), C5.2, J1.6 (Pin_6)
- net U0RXD: now also J1.2 (Pin_2)
- net U0TXD: now also J1.1 (Pin_1)
- net USB_DM_J: now also J1.4 (Pin_4)
- net USB_DP_J: now also J1.3 (Pin_3)
- net 3V3_PWR renamed VOUT
- net VOUT: now also C4.1, TP3.1, U1.6 (VOUT)
- net CFG1_1 renamed CFG1
- net CFG2_1 renamed CFG2
- net CFG3_1 renamed CFG3
- net LX1_1 renamed LX1
- net LX2_1 renamed LX2
- net SNS1_LO renamed SNS_LO
- net VBAT1 renamed VBAT
- net VBAT1_L renamed VBAT_L
- net VBAT1_SENSE renamed VBAT_SENSE
- net VBAT2 renamed VIN
- net VIN: now also C1.1, C2.1, C3.1, Q1.2 (S), U1.1 (EN), U1.10 (VIN), C5.1
- net VBAT2_SENSE: no longer names the net of U4.18 (GPIO4/FSPICLK/ADC1_CH3/MTCK)
- removed net VIN1: C1.1, C2.1, C3.1, Q1.2 (S), TP3.1, U1.1 (EN), U1.10 (VIN), U1.2 (SEL)
- removed net VOUT1: C4.1, TP5.1, U1.6 (VOUT)
- no-connect marks 5 -> 6
Other:
- note added: "3V3 RAIL, SUPERVISOR, RESET"
- note added: "CELL VOLTAGE SENSE (switched 470k/470k divider, ADC1_CH4 on GPIO5)"
- note added: "CR2450 -> P-MOSFET -> TPS63900 (3.3 V) -> VOUT"
- note added: "CR2450 ONLY - NOT RECHARGEABLE. No other supply can reach the rail: the cell is the only energy source. Power-path decision and its limits: docs/decisions.md, docs/power_budget.md (ESTIMATE until measured). Current measurement: remove R1 (cell) or R21 (load) and insert the ammeter. U3 TPS3839K33: 2.93 V typ (2.857-2.974 V), push-pull ~RESET, 200 ms delay; R22 keeps it from fighting SW2 / TP6 (EN)."
- note added: "GPIO8/GPIO9 are strapping pins: GPIO9 low at reset (SW1 held) = download mode. VBAT (pad 15) is tied to 3V3 inside the module (R2 = 0R); connected here as well. Unused GPIO0/1/2/3/4/25: no connect, firmware disables input + pull-down. J1 is a pad row (not fitted) without a supply pin: the cell (or a bench supply on its contacts) powers the board. Reset for programming: SW2 (RST) or the USB-Serial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"
- note added: "SEL = L: VO(1) = 3.3 V (RCFG3 16.2k, table 7-3). Input current limit 100 mA from RCFG1 0R / RCFG2 10.5k (table 7-2; 13.3k = 50 mA option). TI SLVSET3D, +-1 % resistors. C5: 470 uF electrolytic buffer."
- note added: "Switch open: no divider current. GPIO12 high for ~30 ms every 6 h: 470k/470k -> ~3.2 uA while on. The divider top is at the holder terminal (before the 0R link), so a missing cell reads ~0 V."
- note removed: "3V3 RAIL, SUPERVISOR, RESET, DEBUG SUPPLY"
- note removed: "CELL 1: CR2032 -> P-MOSFET -> TPS63900 (3.4 V) -> Schottky -> 3V3_PWR"
- note removed: "CELL 2: CR2032 -> P-MOSFET -> TPS63900 (3.4 V) -> Schottky -> 3V3_PWR"
- note removed: "CELL VOLTAGE SENSE (switched 470k/470k dividers, ADC1_CH0 / ADC1_CH3)"
- note removed: "CR2032 ONLY - NOT RECHARGEABLE. Both cells must be the same brand/lot and replaced together. Power-path decision and its limits: docs/decisions.md, docs/power_budget.md (ESTIMATE until measured). Current measurement: remove R1 / R11 (per cell) or R21 (load) and insert the ammeter. U3 TPS3839K33: 2.93 V typ (2.857-2.974 V), push-pull ~RESET, 200 ms delay; R22 keeps it from fighting SW2 / TP11 (EN)."
- note removed: "GPIO8/GPIO9 are strapping pins: GPIO9 low at reset (SW1 held) = download mode. VBAT (pad 15) is tied to 3V3 inside the module (R2 = 0R); connected here as well. Unused GPIO0/1/2/3/25: no connect, firmware disables input + pull-down. J1 is a pad row (not fitted): pin 6 3V3_DBG only reaches the rail when JP1 is closed. Reset for programming: SW2 (RST) or the USB-Serial/JTAG reset; EN is on test pad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"
- note removed: "SEL = H: VO(2) = 3.4 V (RCFG1 0R), input limit 100 mA (RCFG2 10.5k; 13.3k = 50 mA option), VO(1) = 3.3 V (RCFG3 16.2k, unused). TI SLVSET3D tables 7-2/7-3, +-1 % resistors."
- note removed: "Switches open: no divider current. GPIO12 high for ~30 ms every 6 h: 470k/470k -> 3.3 uA per cell. Each divider top is at the holder terminal (before the 0R link), so a missing cell reads ~0 V."
- moved on the sheet: C1, C2, C3, R2, R3, R4
